Commit message: Update xarm_ros2 submodule for gripper mesh

File: xarm_description/urdf/gripper/xarm_gripper.urdf.xacro (robot description, xacro)
@@ -60,13 +60,17 @@
           iyy="1.7225E-05" iyz="4.6433E-06" izz="5.1466E-06" />
       </inertial>
-      <xacro:common_link_visual
-        mesh_filename="gripper/xarm/left_finger"
-        origin_xyz="0 0 0"
-        origin_rpy="0 0 0"
-        material_name="${prefix}Silver" />
-      <xacro:common_link_collision
-        mesh_filename="gripper/xarm/left_finger"
-        origin_xyz="0 0 0"
-        origin_rpy="0 0 0" />
+      <visual>
+        <origin xyz="0 0 0" rpy="0 0 0"/>
+        <geometry>
+          <mesh filename="${mesh_path}/gripper/xarm/queeenb_left_finger.stl" scale="0.001 0.001 0.001"/>
+        </geometry>
+        <material name="${prefix}Silver"/>
+      </visual>
+      <collision>
+        <origin xyz="0 0 0" rpy="0 0 0"/>
+        <geometry>
+          <mesh filename="${mesh_path}/gripper/xarm/queeenb_left_finger.stl" scale="0.001 0.001 0.001"/>
+        </geometry>
+      </collision>
     </link>
     <joint name="${prefix}left_finger_joint" type="revolute">
@@ -138,13 +142,17 @@
           iyy="1.7225E-05" iyz="-4.6435E-06" izz="5.1466E-06" />
       </inertial>
-      <xacro:common_link_visual
-        mesh_filename="gripper/xarm/right_finger"
-        origin_xyz="0 0 0"
-        origin_rpy="0 0 0"
-        material_name="${prefix}Silver" />
-      <xacro:common_link_collision
-        mesh_filename="gripper/xarm/right_finger"
-        origin_xyz="0 0 0"
-        origin_rpy="0 0 0" />
+      <visual>
+        <origin xyz="0 0 0" rpy="0 0 0"/>
+        <geometry>
+          <mesh filename="${mesh_path}/gripper/xarm/queeenb_right_finger.stl" scale="0.001 0.001 0.001"/>
+        </geometry>
+        <material name="${prefix}Silver"/>
+      </visual>
+      <collision>
+        <origin xyz="0 0 0" rpy="0 0 0"/>
+        <geometry>
+          <mesh filename="${mesh_path}/gripper/xarm/queeenb_right_finger.stl" scale="0.001 0.001 0.001"/>
+        </geometry>
+      </collision>
     </link>
     <joint name="${prefix}right_finger_joint" type="revolute">

Commit message: Update xArm gripper finger angle

File: xarm_description/urdf/gripper/xarm_gripper.urdf.xacro (robot description, xacro)
@@ -61,5 +61,5 @@
       </inertial>
       <visual>
-        <origin xyz="0 0 0" rpy="0 0 0"/>
+        <origin xyz="0 0 0" rpy="0 0 1.5707963267948966"/>
         <geometry>
           <mesh filename="${mesh_path}/gripper/xarm/queeenb_left_finger.stl" scale="0.001 0.001 0.001"/>
@@ -68,5 +68,5 @@
       </visual>
       <collision>
-        <origin xyz="0 0 0" rpy="0 0 0"/>
+        <origin xyz="0 0 0" rpy="0 0 1.5707963267948966"/>
         <geometry>
           <mesh filename="${mesh_path}/gripper/xarm/queeenb_left_finger.stl" scale="0.001 0.001 0.001"/>
@@ -143,5 +143,5 @@
       </inertial>
       <visual>
-        <origin xyz="0 0 0" rpy="0 0 0"/>
+        <origin xyz="0 0 0" rpy="0 0 1.5707963267948966"/>
         <geometry>
           <mesh filename="${mesh_path}/gripper/xarm/queeenb_right_finger.stl" scale="0.001 0.001 0.001"/>
@@ -150,5 +150,5 @@
       </visual>
       <collision>
-        <origin xyz="0 0 0" rpy="0 0 0"/>
+        <origin xyz="0 0 0" rpy="0 0 1.5707963267948966"/>
         <geometry>
           <mesh filename="${mesh_path}/gripper/xarm/queeenb_right_finger.stl" scale="0.001 0.001 0.001"/>

Commit message: Update xArm gripper finger angle

File: xarm_description/urdf/gripper/xarm_gripper.urdf.xacro (robot description, xacro)
@@ -63,5 +63,5 @@
         <origin xyz="0 0 0" rpy="0 0 1.5707963267948966"/>
         <geometry>
-          <mesh filename="${mesh_path}/gripper/xarm/queeenb_left_finger.stl" scale="0.001 0.001 0.001"/>
+          <mesh filename="${mesh_path}/gripper/xarm/queeenb_right_finger.stl" scale="0.001 0.001 0.001"/>
         </geometry>
         <material name="${prefix}Silver"/>
@@ -70,5 +70,5 @@
         <origin xyz="0 0 0" rpy="0 0 1.5707963267948966"/>
         <geometry>
-          <mesh filename="${mesh_path}/gripper/xarm/queeenb_left_finger.stl" scale="0.001 0.001 0.001"/>
+          <mesh filename="${mesh_path}/gripper/xarm/queeenb_right_finger.stl" scale="0.001 0.001 0.001"/>
         </geometry>
       </collision>
@@ -145,5 +145,5 @@
         <origin xyz="0 0 0" rpy="0 0 1.5707963267948966"/>
         <geometry>
-          <mesh filename="${mesh_path}/gripper/xarm/queeenb_right_finger.stl" scale="0.001 0.001 0.001"/>
+          <mesh filename="${mesh_path}/gripper/xarm/queeenb_left_finger.stl" scale="0.001 0.001 0.001"/>
         </geometry>
         <material name="${prefix}Silver"/>
@@ -152,5 +152,5 @@
         <origin xyz="0 0 0" rpy="0 0 1.5707963267948966"/>
         <geometry>
-          <mesh filename="${mesh_path}/gripper/xarm/queeenb_right_finger.stl" scale="0.001 0.001 0.001"/>
+          <mesh filename="${mesh_path}/gripper/xarm/queeenb_left_finger.stl" scale="0.001 0.001 0.001"/>
         </geometry>
       </collision>

Commit message: Update xArm gripper finger angle

File: xarm_description/urdf/gripper/xarm_gripper.urdf.xacro (robot description, xacro)
@@ -61,5 +61,5 @@
       </inertial>
       <visual>
-        <origin xyz="0 0 0" rpy="0 0 1.5707963267948966"/>
+        <origin xyz="0 0 0" rpy="3.141592653589793 0 1.5707963267948966"/>
         <geometry>
           <mesh filename="${mesh_path}/gripper/xarm/queeenb_right_finger.stl" scale="0.001 0.001 0.001"/>
@@ -68,5 +68,5 @@
       </visual>
       <collision>
-        <origin xyz="0 0 0" rpy="0 0 1.5707963267948966"/>
+        <origin xyz="0 0 0" rpy="3.141592653589793 0 1.5707963267948966"/>
         <geometry>
           <mesh filename="${mesh_path}/gripper/xarm/queeenb_right_finger.stl" scale="0.001 0.001 0.001"/>
@@ -143,5 +143,5 @@
       </inertial>
       <visual>
-        <origin xyz="0 0 0" rpy="0 0 1.5707963267948966"/>
+        <origin xyz="0 0 0" rpy="3.141592653589793 0 1.5707963267948966"/>
         <geometry>
           <mesh filename="${mesh_path}/gripper/xarm/queeenb_left_finger.stl" scale="0.001 0.001 0.001"/>
@@ -150,5 +150,5 @@
       </visual>
       <collision>
-        <origin xyz="0 0 0" rpy="0 0 1.5707963267948966"/>
+        <origin xyz="0 0 0" rpy="3.141592653589793 0 1.5707963267948966"/>
         <geometry>
           <mesh filename="${mesh_path}/gripper/xarm/queeenb_left_finger.stl" scale="0.001 0.001 0.001"/>

Commit message: Update xarm_ros2 submodule for gripper mesh position

File: xarm_description/urdf/gripper/xarm_gripper.urdf.xacro (robot description, xacro)
@@ -61,5 +61,5 @@
       </inertial>
       <visual>
-        <origin xyz="0 0 0" rpy="3.141592653589793 0 1.5707963267948966"/>
+        <origin xyz="0.0675 -0.0375 0.010" rpy="3.141592653589793 0 1.5707963267948966"/>
         <geometry>
           <mesh filename="${mesh_path}/gripper/xarm/queeenb_right_finger.stl" scale="0.001 0.001 0.001"/>
@@ -68,5 +68,5 @@
       </visual>
       <collision>
-        <origin xyz="0 0 0" rpy="3.141592653589793 0 1.5707963267948966"/>
+        <origin xyz="0.0675 -0.0375 0.010" rpy="3.141592653589793 0 1.5707963267948966"/>
         <geometry>
           <mesh filename="${mesh_path}/gripper/xarm/queeenb_right_finger.stl" scale="0.001 0.001 0.001"/>
@@ -143,5 +143,5 @@
       </inertial>
       <visual>
-        <origin xyz="0 0 0" rpy="3.141592653589793 0 1.5707963267948966"/>
+        <origin xyz="0.0675 0.0375 0.010" rpy="3.141592653589793 0 1.5707963267948966"/>
         <geometry>
           <mesh filename="${mesh_path}/gripper/xarm/queeenb_left_finger.stl" scale="0.001 0.001 0.001"/>
@@ -150,5 +150,5 @@
       </visual>
       <collision>
-        <origin xyz="0 0 0" rpy="3.141592653589793 0 1.5707963267948966"/>
+        <origin xyz="0.0675 0.0375 0.010" rpy="3.141592653589793 0 1.5707963267948966"/>
         <geometry>
           <mesh filename="${mesh_path}/gripper/xarm/queeenb_left_finger.stl" scale="0.001 0.001 0.001"/>

Commit message: Update xarm_ros2 submodule for gripper mesh position

File: xarm_description/urdf/gripper/xarm_gripper.urdf.xacro (robot description, xacro)
@@ -60,6 +60,15 @@
           iyy="1.7225E-05" iyz="4.6433E-06" izz="5.1466E-06" />
       </inertial>
+      <xacro:common_link_visual
+        mesh_filename="gripper/xarm/left_finger"
+        origin_xyz="0 0 0"
+        origin_rpy="0 0 0"
+        material_name="${prefix}Silver" />
+      <xacro:common_link_collision
+        mesh_filename="gripper/xarm/left_finger"
+        origin_xyz="0 0 0"
+        origin_rpy="0 0 0" />
       <visual>
-        <origin xyz="0.0675 -0.0375 0.010" rpy="3.141592653589793 0 1.5707963267948966"/>
+        <origin xyz="0.0675 -0.0475 0.071" rpy="3.141592653589793 0 1.5707963267948966"/>
         <geometry>
           <mesh filename="${mesh_path}/gripper/xarm/queeenb_right_finger.stl" scale="0.001 0.001 0.001"/>
@@ -68,5 +77,5 @@
       </visual>
       <collision>
-        <origin xyz="0.0675 -0.0375 0.010" rpy="3.141592653589793 0 1.5707963267948966"/>
+        <origin xyz="0.0675 -0.0475 0.071" rpy="3.141592653589793 0 1.5707963267948966"/>
         <geometry>
           <mesh filename="${mesh_path}/gripper/xarm/queeenb_right_finger.stl" scale="0.001 0.001 0.001"/>
@@ -142,6 +151,15 @@
           iyy="1.7225E-05" iyz="-4.6435E-06" izz="5.1466E-06" />
       </inertial>
+      <xacro:common_link_visual
+        mesh_filename="gripper/xarm/right_finger"
+        origin_xyz="0 0 0"
+        origin_rpy="0 0 0"
+        material_name="${prefix}Silver" />
+      <xacro:common_link_collision
+        mesh_filename="gripper/xarm/right_finger"
+        origin_xyz="0 0 0"
+        origin_rpy="0 0 0" />
       <visual>
-        <origin xyz="0.0675 0.0375 0.010" rpy="3.141592653589793 0 1.5707963267948966"/>
+        <origin xyz="0.0675 0.0475 0.071" rpy="3.141592653589793 0 1.5707963267948966"/>
         <geometry>
           <mesh filename="${mesh_path}/gripper/xarm/queeenb_left_finger.stl" scale="0.001 0.001 0.001"/>
@@ -150,5 +168,5 @@
       </visual>
       <collision>
-        <origin xyz="0.0675 0.0375 0.010" rpy="3.141592653589793 0 1.5707963267948966"/>
+        <origin xyz="0.0675 0.0475 0.071" rpy="3.141592653589793 0 1.5707963267948966"/>
         <geometry>
           <mesh filename="${mesh_path}/gripper/xarm/queeenb_left_finger.stl" scale="0.001 0.001 0.001"/>

Commit message: Update xarm_ros2 submodule for gripper mesh

File: xarm_description/urdf/gripper/xarm_gripper.urdf.xacro (robot description, xacro)
@@ -70,5 +70,5 @@
         origin_rpy="0 0 0" />
       <visual>
-        <origin xyz="0.0675 -0.0475 0.071" rpy="3.141592653589793 0 1.5707963267948966"/>
+        <origin xyz="0.0400 -0.0220 0.0450" rpy="3.141592653589793 0 1.5707963267948966"/>
         <geometry>
           <mesh filename="${mesh_path}/gripper/xarm/queeenb_right_finger.stl" scale="0.001 0.001 0.001"/>
@@ -77,5 +77,5 @@
       </visual>
       <collision>
-        <origin xyz="0.0675 -0.0475 0.071" rpy="3.141592653589793 0 1.5707963267948966"/>
+        <origin xyz="0.0400 -0.0220 0.0450" rpy="3.141592653589793 0 1.5707963267948966"/>
         <geometry>
           <mesh filename="${mesh_path}/gripper/xarm/queeenb_right_finger.stl" scale="0.001 0.001 0.001"/>
@@ -161,5 +161,5 @@
         origin_rpy="0 0 0" />
       <visual>
-        <origin xyz="0.0675 0.0475 0.071" rpy="3.141592653589793 0 1.5707963267948966"/>
+        <origin xyz="0.0400 0.0220 0.0450" rpy="3.141592653589793 0 1.5707963267948966"/>
         <geometry>
           <mesh filename="${mesh_path}/gripper/xarm/queeenb_left_finger.stl" scale="0.001 0.001 0.001"/>
@@ -168,5 +168,5 @@
       </visual>
       <collision>
-        <origin xyz="0.0675 0.0475 0.071" rpy="3.141592653589793 0 1.5707963267948966"/>
+        <origin xyz="0.0400 0.0220 0.0450" rpy="3.141592653589793 0 1.5707963267948966"/>
         <geometry>
           <mesh filename="${mesh_path}/gripper/xarm/queeenb_left_finger.stl" scale="0.001 0.001 0.001"/>

Commit message: Update xarm_ros2 submodule for gripper mesh

File: xarm_description/urdf/gripper/xarm_gripper.urdf.xacro (robot description, xacro)
@@ -70,5 +70,5 @@
         origin_rpy="0 0 0" />
       <visual>
-        <origin xyz="0.0400 -0.0220 0.0450" rpy="3.141592653589793 0 1.5707963267948966"/>
+        <origin xyz="0.0400 -0.0060 0.0100" rpy="3.141592653589793 0 1.5707963267948966"/>
         <geometry>
           <mesh filename="${mesh_path}/gripper/xarm/queeenb_right_finger.stl" scale="0.001 0.001 0.001"/>
@@ -77,5 +77,5 @@
       </visual>
       <collision>
-        <origin xyz="0.0400 -0.0220 0.0450" rpy="3.141592653589793 0 1.5707963267948966"/>
+        <origin xyz="0.0400 -0.0060 0.0100" rpy="3.141592653589793 0 1.5707963267948966"/>
         <geometry>
           <mesh filename="${mesh_path}/gripper/xarm/queeenb_right_finger.stl" scale="0.001 0.001 0.001"/>
@@ -161,5 +161,5 @@
         origin_rpy="0 0 0" />
       <visual>
-        <origin xyz="0.0400 0.0220 0.0450" rpy="3.141592653589793 0 1.5707963267948966"/>
+        <origin xyz="0.0400 0.0060 0.0100" rpy="3.141592653589793 0 1.5707963267948966"/>
         <geometry>
           <mesh filename="${mesh_path}/gripper/xarm/queeenb_left_finger.stl" scale="0.001 0.001 0.001"/>
@@ -168,5 +168,5 @@
       </visual>
       <collision>
-        <origin xyz="0.0400 0.0220 0.0450" rpy="3.141592653589793 0 1.5707963267948966"/>
+        <origin xyz="0.0400 0.0060 0.0100" rpy="3.141592653589793 0 1.5707963267948966"/>
         <geometry>
           <mesh filename="${mesh_path}/gripper/xarm/queeenb_left_finger.stl" scale="0.001 0.001 0.001"/>

Commit message: Update xarm_ros2 submodule for gripper mesh

File: xarm_description/urdf/gripper/xarm_gripper.urdf.xacro (robot description, xacro)
@@ -70,5 +70,5 @@
         origin_rpy="0 0 0" />
       <visual>
-        <origin xyz="0.0400 -0.0060 0.0100" rpy="3.141592653589793 0 1.5707963267948966"/>
+        <origin xyz="0.0400 -0.0500 0.0180" rpy="3.141592653589793 0 1.5707963267948966"/>
         <geometry>
           <mesh filename="${mesh_path}/gripper/xarm/queeenb_right_finger.stl" scale="0.001 0.001 0.001"/>
@@ -77,5 +77,5 @@
       </visual>
       <collision>
-        <origin xyz="0.0400 -0.0060 0.0100" rpy="3.141592653589793 0 1.5707963267948966"/>
+        <origin xyz="0.0400 -0.0500 0.0180" rpy="3.141592653589793 0 1.5707963267948966"/>
         <geometry>
           <mesh filename="${mesh_path}/gripper/xarm/queeenb_right_finger.stl" scale="0.001 0.001 0.001"/>
@@ -161,5 +161,5 @@
         origin_rpy="0 0 0" />
       <visual>
-        <origin xyz="0.0400 0.0060 0.0100" rpy="3.141592653589793 0 1.5707963267948966"/>
+        <origin xyz="0.0400 0.0500 0.0180" rpy="3.141592653589793 0 1.5707963267948966"/>
         <geometry>
           <mesh filename="${mesh_path}/gripper/xarm/queeenb_left_finger.stl" scale="0.001 0.001 0.001"/>
@@ -168,5 +168,5 @@
       </visual>
       <collision>
-        <origin xyz="0.0400 0.0060 0.0100" rpy="3.141592653589793 0 1.5707963267948966"/>
+        <origin xyz="0.0400 0.0500 0.0180" rpy="3.141592653589793 0 1.5707963267948966"/>
         <geometry>
           <mesh filename="${mesh_path}/gripper/xarm/queeenb_left_finger.stl" scale="0.001 0.001 0.001"/>

Commit message: Update xarm_ros2 submodule for gripper mesh position

File: xarm_description/urdf/gripper/xarm_gripper.urdf.xacro (robot description, xacro)
@@ -70,5 +70,5 @@
         origin_rpy="0 0 0" />
       <visual>
-        <origin xyz="0.0400 -0.0500 0.0180" rpy="3.141592653589793 0 1.5707963267948966"/>
+        <origin xyz="0.0400 -0.0500 -0.0280" rpy="3.141592653589793 0 1.5707963267948966"/>
         <geometry>
           <mesh filename="${mesh_path}/gripper/xarm/queeenb_right_finger.stl" scale="0.001 0.001 0.001"/>
@@ -77,5 +77,5 @@
       </visual>
       <collision>
-        <origin xyz="0.0400 -0.0500 0.0180" rpy="3.141592653589793 0 1.5707963267948966"/>
+        <origin xyz="0.0400 -0.0500 -0.0280" rpy="3.141592653589793 0 1.5707963267948966"/>
         <geometry>
           <mesh filename="${mesh_path}/gripper/xarm/queeenb_right_finger.stl" scale="0.001 0.001 0.001"/>
@@ -161,5 +161,5 @@
         origin_rpy="0 0 0" />
       <visual>
-        <origin xyz="0.0400 0.0500 0.0180" rpy="3.141592653589793 0 1.5707963267948966"/>
+        <origin xyz="0.0400 0.0500 -0.0280" rpy="3.141592653589793 0 1.5707963267948966"/>
         <geometry>
           <mesh filename="${mesh_path}/gripper/xarm/queeenb_left_finger.stl" scale="0.001 0.001 0.001"/>
@@ -168,5 +168,5 @@
       </visual>
       <collision>
-        <origin xyz="0.0400 0.0500 0.0180" rpy="3.141592653589793 0 1.5707963267948966"/>
+        <origin xyz="0.0400 0.0500 -0.0280" rpy="3.141592653589793 0 1.5707963267948966"/>
         <geometry>
           <mesh filename="${mesh_path}/gripper/xarm/queeenb_left_finger.stl" scale="0.001 0.001 0.001"/>

Commit message: Update xarm_ros2 submodule for gripper mesh position

File: xarm_description/urdf/gripper/xarm_gripper.urdf.xacro (robot description, xacro)
@@ -70,5 +70,5 @@
         origin_rpy="0 0 0" />
       <visual>
-        <origin xyz="0.0400 -0.0500 -0.0280" rpy="3.141592653589793 0 1.5707963267948966"/>
+        <origin xyz="0.0400 -0.0500 0.0600" rpy="3.141592653589793 0 1.5707963267948966"/>
         <geometry>
           <mesh filename="${mesh_path}/gripper/xarm/queeenb_right_finger.stl" scale="0.001 0.001 0.001"/>
@@ -77,5 +77,5 @@
       </visual>
       <collision>
-        <origin xyz="0.0400 -0.0500 -0.0280" rpy="3.141592653589793 0 1.5707963267948966"/>
+        <origin xyz="0.0400 -0.0500 0.0600" rpy="3.141592653589793 0 1.5707963267948966"/>
         <geometry>
           <mesh filename="${mesh_path}/gripper/xarm/queeenb_right_finger.stl" scale="0.001 0.001 0.001"/>
@@ -161,5 +161,5 @@
         origin_rpy="0 0 0" />
       <visual>
-        <origin xyz="0.0400 0.0500 -0.0280" rpy="3.141592653589793 0 1.5707963267948966"/>
+        <origin xyz="0.0400 0.0500 0.0600" rpy="3.141592653589793 0 1.5707963267948966"/>
         <geometry>
           <mesh filename="${mesh_path}/gripper/xarm/queeenb_left_finger.stl" scale="0.001 0.001 0.001"/>
@@ -168,5 +168,5 @@
       </visual>
       <collision>
-        <origin xyz="0.0400 0.0500 -0.0280" rpy="3.141592653589793 0 1.5707963267948966"/>
+        <origin xyz="0.0400 0.0500 0.0600" rpy="3.141592653589793 0 1.5707963267948966"/>
         <geometry>
           <mesh filename="${mesh_path}/gripper/xarm/queeenb_left_finger.stl" scale="0.001 0.001 0.001"/>

Commit message: Update xarm_ros2 submodule for gripper mesh position

File: xarm_description/urdf/gripper/xarm_gripper.urdf.xacro (robot description, xacro)
@@ -70,5 +70,5 @@
         origin_rpy="0 0 0" />
       <visual>
-        <origin xyz="0.0400 -0.0500 0.0600" rpy="3.141592653589793 0 1.5707963267948966"/>
+        <origin xyz="0.0400 -0.0500 0.0800" rpy="3.141592653589793 0 1.5707963267948966"/>
         <geometry>
           <mesh filename="${mesh_path}/gripper/xarm/queeenb_right_finger.stl" scale="0.001 0.001 0.001"/>

Commit message: Update xarm_ros2 submodule for gripper mesh position(origin z = 0.1100)

File: xarm_description/urdf/gripper/xarm_gripper.urdf.xacro (robot description, xacro)
@@ -70,5 +70,5 @@
         origin_rpy="0 0 0" />
       <visual>
-        <origin xyz="0.0400 -0.0500 0.0800" rpy="3.141592653589793 0 1.5707963267948966"/>
+        <origin xyz="0.0400 -0.0500 0.1100" rpy="3.141592653589793 0 1.5707963267948966"/>
         <geometry>
           <mesh filename="${mesh_path}/gripper/xarm/queeenb_right_finger.stl" scale="0.001 0.001 0.001"/>
@@ -77,5 +77,5 @@
       </visual>
       <collision>
-        <origin xyz="0.0400 -0.0500 0.0600" rpy="3.141592653589793 0 1.5707963267948966"/>
+        <origin xyz="0.0400 -0.0500 0.1100" rpy="3.141592653589793 0 1.5707963267948966"/>
         <geometry>
           <mesh filename="${mesh_path}/gripper/xarm/queeenb_right_finger.stl" scale="0.001 0.001 0.001"/>
@@ -161,5 +161,5 @@
         origin_rpy="0 0 0" />
       <visual>
-        <origin xyz="0.0400 0.0500 0.0600" rpy="3.141592653589793 0 1.5707963267948966"/>
+        <origin xyz="0.0400 0.0500 0.1100" rpy="3.141592653589793 0 1.5707963267948966"/>
         <geometry>
           <mesh filename="${mesh_path}/gripper/xarm/queeenb_left_finger.stl" scale="0.001 0.001 0.001"/>
@@ -168,5 +168,5 @@
       </visual>
       <collision>
-        <origin xyz="0.0400 0.0500 0.0600" rpy="3.141592653589793 0 1.5707963267948966"/>
+        <origin xyz="0.0400 0.0500 0.1100" rpy="3.141592653589793 0 1.5707963267948966"/>
         <geometry>
           <mesh filename="${mesh_path}/gripper/xarm/queeenb_left_finger.stl" scale="0.001 0.001 0.001"/>

Commit message: Update xarm_ros2 submodule for gripper mesh position(origin x=0.0550)

File: xarm_description/urdf/gripper/xarm_gripper.urdf.xacro (robot description, xacro)
@@ -70,5 +70,5 @@
         origin_rpy="0 0 0" />
       <visual>
-        <origin xyz="0.0400 -0.0500 0.1100" rpy="3.141592653589793 0 1.5707963267948966"/>
+        <origin xyz="0.0550 -0.0500 0.1100" rpy="3.141592653589793 0 1.5707963267948966"/>
         <geometry>
           <mesh filename="${mesh_path}/gripper/xarm/queeenb_right_finger.stl" scale="0.001 0.001 0.001"/>
@@ -77,5 +77,5 @@
       </visual>
       <collision>
-        <origin xyz="0.0400 -0.0500 0.1100" rpy="3.141592653589793 0 1.5707963267948966"/>
+        <origin xyz="0.0550 -0.0500 0.1100" rpy="3.141592653589793 0 1.5707963267948966"/>
         <geometry>
           <mesh filename="${mesh_path}/gripper/xarm/queeenb_right_finger.stl" scale="0.001 0.001 0.001"/>
@@ -161,5 +161,5 @@
         origin_rpy="0 0 0" />
       <visual>
-        <origin xyz="0.0400 0.0500 0.1100" rpy="3.141592653589793 0 1.5707963267948966"/>
+        <origin xyz="0.0550 0.0500 0.1100" rpy="3.141592653589793 0 1.5707963267948966"/>
         <geometry>
           <mesh filename="${mesh_path}/gripper/xarm/queeenb_left_finger.stl" scale="0.001 0.001 0.001"/>
@@ -168,5 +168,5 @@
       </visual>
       <collision>
-        <origin xyz="0.0400 0.0500 0.1100" rpy="3.141592653589793 0 1.5707963267948966"/>
+        <origin xyz="0.0550 0.0500 0.1100" rpy="3.141592653589793 0 1.5707963267948966"/>
         <geometry>
           <mesh filename="${mesh_path}/gripper/xarm/queeenb_left_finger.stl" scale="0.001 0.001 0.001"/>
