Commit message: Update xarm_ros2 submodule for gripper mesh position(origin x=0.020)

File: xarm_description/urdf/gripper/xarm_gripper.urdf.xacro (robot description, xacro)
@@ -70,5 +70,5 @@
         origin_rpy="0 0 0" />
       <visual>
-        <origin xyz="0.0550 -0.0500 0.1100" rpy="3.141592653589793 0 1.5707963267948966"/>
+        <origin xyz="0.0200 -0.0500 0.1100" rpy="3.141592653589793 0 1.5707963267948966"/>
         <geometry>
           <mesh filename="${mesh_path}/gripper/xarm/queeenb_right_finger.stl" scale="0.001 0.001 0.001"/>
@@ -77,5 +77,5 @@
       </visual>
       <collision>
-        <origin xyz="0.0550 -0.0500 0.1100" rpy="3.141592653589793 0 1.5707963267948966"/>
+        <origin xyz="0.0200 -0.0500 0.1100" rpy="3.141592653589793 0 1.5707963267948966"/>
         <geometry>
           <mesh filename="${mesh_path}/gripper/xarm/queeenb_right_finger.stl" scale="0.001 0.001 0.001"/>
@@ -161,5 +161,5 @@
         origin_rpy="0 0 0" />
       <visual>
-        <origin xyz="0.0550 0.0500 0.1100" rpy="3.141592653589793 0 1.5707963267948966"/>
+        <origin xyz="0.0200 0.0500 0.1100" rpy="3.141592653589793 0 1.5707963267948966"/>
         <geometry>
           <mesh filename="${mesh_path}/gripper/xarm/queeenb_left_finger.stl" scale="0.001 0.001 0.001"/>
@@ -168,5 +168,5 @@
       </visual>
       <collision>
-        <origin xyz="0.0550 0.0500 0.1100" rpy="3.141592653589793 0 1.5707963267948966"/>
+        <origin xyz="0.0200 0.0500 0.1100" rpy="3.141592653589793 0 1.5707963267948966"/>
         <geometry>
           <mesh filename="${mesh_path}/gripper/xarm/queeenb_left_finger.stl" scale="0.001 0.001 0.001"/>

Commit message: Update xarm_ros2 submodule for gripper mesh position(origin x=0.030)

File: xarm_description/urdf/gripper/xarm_gripper.urdf.xacro (robot description, xacro)
@@ -70,5 +70,5 @@
         origin_rpy="0 0 0" />
       <visual>
-        <origin xyz="0.0200 -0.0500 0.1100" rpy="3.141592653589793 0 1.5707963267948966"/>
+        <origin xyz="0.0300 -0.0500 0.1100" rpy="3.141592653589793 0 1.5707963267948966"/>
         <geometry>
           <mesh filename="${mesh_path}/gripper/xarm/queeenb_right_finger.stl" scale="0.001 0.001 0.001"/>
@@ -77,5 +77,5 @@
       </visual>
       <collision>
-        <origin xyz="0.0200 -0.0500 0.1100" rpy="3.141592653589793 0 1.5707963267948966"/>
+        <origin xyz="0.0300 -0.0500 0.1100" rpy="3.141592653589793 0 1.5707963267948966"/>
         <geometry>
           <mesh filename="${mesh_path}/gripper/xarm/queeenb_right_finger.stl" scale="0.001 0.001 0.001"/>
@@ -161,5 +161,5 @@
         origin_rpy="0 0 0" />
       <visual>
-        <origin xyz="0.0200 0.0500 0.1100" rpy="3.141592653589793 0 1.5707963267948966"/>
+        <origin xyz="0.0300 0.0500 0.1100" rpy="3.141592653589793 0 1.5707963267948966"/>
         <geometry>
           <mesh filename="${mesh_path}/gripper/xarm/queeenb_left_finger.stl" scale="0.001 0.001 0.001"/>
@@ -168,5 +168,5 @@
       </visual>
       <collision>
-        <origin xyz="0.0200 0.0500 0.1100" rpy="3.141592653589793 0 1.5707963267948966"/>
+        <origin xyz="0.0300 0.0500 0.1100" rpy="3.141592653589793 0 1.5707963267948966"/>
         <geometry>
           <mesh filename="${mesh_path}/gripper/xarm/queeenb_left_finger.stl" scale="0.001 0.001 0.001"/>
