Commit message: Replace gripper fingertip mesh with Gripper v2

File: xarm_description/urdf/gripper/xarm_gripper.urdf.xacro (robot description, xacro)
@@ -70,14 +70,14 @@
         origin_rpy="0 0 0" />
       <visual>
-        <origin xyz="0.0300 -0.0500 0.1100" rpy="3.141592653589793 0 1.5707963267948966"/>
-        <geometry>
-          <mesh filename="${mesh_path}/gripper/xarm/queeenb_right_finger.stl" scale="0.001 0.001 0.001"/>
+        <origin xyz="0.045 -0.048 0.096" rpy="1.5707963267948966 0 -1.5707963267948966"/>
+        <geometry>
+          <mesh filename="${mesh_path}/gripper/xarm/queeenb_gripper_v2_left.stl" scale="0.001 0.001 0.001"/>
         </geometry>
         <material name="${prefix}Silver"/>
       </visual>
       <collision>
-        <origin xyz="0.0300 -0.0500 0.1100" rpy="3.141592653589793 0 1.5707963267948966"/>
-        <geometry>
-          <mesh filename="${mesh_path}/gripper/xarm/queeenb_right_finger.stl" scale="0.001 0.001 0.001"/>
+        <origin xyz="0.045 -0.048 0.096" rpy="1.5707963267948966 0 -1.5707963267948966"/>
+        <geometry>
+          <mesh filename="${mesh_path}/gripper/xarm/queeenb_gripper_v2_left.stl" scale="0.001 0.001 0.001"/>
         </geometry>
       </collision>
@@ -161,14 +161,14 @@
         origin_rpy="0 0 0" />
       <visual>
-        <origin xyz="0.0300 0.0500 0.1100" rpy="3.141592653589793 0 1.5707963267948966"/>
-        <geometry>
-          <mesh filename="${mesh_path}/gripper/xarm/queeenb_left_finger.stl" scale="0.001 0.001 0.001"/>
+        <origin xyz="0.045 0.048 0.096" rpy="1.5707963267948966 0 1.5707963267948966"/>
+        <geometry>
+          <mesh filename="${mesh_path}/gripper/xarm/queeenb_gripper_v2_right.stl" scale="0.001 0.001 0.001"/>
         </geometry>
         <material name="${prefix}Silver"/>
       </visual>
       <collision>
-        <origin xyz="0.0300 0.0500 0.1100" rpy="3.141592653589793 0 1.5707963267948966"/>
-        <geometry>
-          <mesh filename="${mesh_path}/gripper/xarm/queeenb_left_finger.stl" scale="0.001 0.001 0.001"/>
+        <origin xyz="0.045 0.048 0.096" rpy="1.5707963267948966 0 1.5707963267948966"/>
+        <geometry>
+          <mesh filename="${mesh_path}/gripper/xarm/queeenb_gripper_v2_right.stl" scale="0.001 0.001 0.001"/>
         </geometry>
       </collision>

Commit message: Swap gripper v2 fingertip left/right so paddles face the near side

File: xarm_description/urdf/gripper/xarm_gripper.urdf.xacro (robot description, xacro)
@@ -70,14 +70,14 @@
         origin_rpy="0 0 0" />
       <visual>
-        <origin xyz="0.045 -0.048 0.096" rpy="1.5707963267948966 0 -1.5707963267948966"/>
-        <geometry>
-          <mesh filename="${mesh_path}/gripper/xarm/queeenb_gripper_v2_left.stl" scale="0.001 0.001 0.001"/>
+        <origin xyz="-0.045 -0.048 0.096" rpy="1.5707963267948966 0 -1.5707963267948966"/>
+        <geometry>
+          <mesh filename="${mesh_path}/gripper/xarm/queeenb_gripper_v2_right.stl" scale="0.001 0.001 0.001"/>
         </geometry>
         <material name="${prefix}Silver"/>
       </visual>
       <collision>
-        <origin xyz="0.045 -0.048 0.096" rpy="1.5707963267948966 0 -1.5707963267948966"/>
-        <geometry>
-          <mesh filename="${mesh_path}/gripper/xarm/queeenb_gripper_v2_left.stl" scale="0.001 0.001 0.001"/>
+        <origin xyz="-0.045 -0.048 0.096" rpy="1.5707963267948966 0 -1.5707963267948966"/>
+        <geometry>
+          <mesh filename="${mesh_path}/gripper/xarm/queeenb_gripper_v2_right.stl" scale="0.001 0.001 0.001"/>
         </geometry>
       </collision>
@@ -161,14 +161,14 @@
         origin_rpy="0 0 0" />
       <visual>
-        <origin xyz="0.045 0.048 0.096" rpy="1.5707963267948966 0 1.5707963267948966"/>
-        <geometry>
-          <mesh filename="${mesh_path}/gripper/xarm/queeenb_gripper_v2_right.stl" scale="0.001 0.001 0.001"/>
+        <origin xyz="-0.045 0.048 0.096" rpy="1.5707963267948966 0 1.5707963267948966"/>
+        <geometry>
+          <mesh filename="${mesh_path}/gripper/xarm/queeenb_gripper_v2_left.stl" scale="0.001 0.001 0.001"/>
         </geometry>
         <material name="${prefix}Silver"/>
       </visual>
       <collision>
-        <origin xyz="0.045 0.048 0.096" rpy="1.5707963267948966 0 1.5707963267948966"/>
-        <geometry>
-          <mesh filename="${mesh_path}/gripper/xarm/queeenb_gripper_v2_right.stl" scale="0.001 0.001 0.001"/>
+        <origin xyz="-0.045 0.048 0.096" rpy="1.5707963267948966 0 1.5707963267948966"/>
+        <geometry>
+          <mesh filename="${mesh_path}/gripper/xarm/queeenb_gripper_v2_left.stl" scale="0.001 0.001 0.001"/>
         </geometry>
       </collision>

Commit message: Update gripper mesh and pose

File: xarm_description/urdf/gripper/xarm_gripper.urdf.xacro (robot description, xacro)
@@ -70,14 +70,14 @@
         origin_rpy="0 0 0" />
       <visual>
-        <origin xyz="-0.045 -0.048 0.096" rpy="1.5707963267948966 0 -1.5707963267948966"/>
-        <geometry>
-          <mesh filename="${mesh_path}/gripper/xarm/queeenb_gripper_v2_right.stl" scale="0.001 0.001 0.001"/>
+        <origin xyz="0.045 -0.048 0.096" rpy="1.5707963267948966 0 -1.5707963267948966"/>
+        <geometry>
+          <mesh filename="${mesh_path}/gripper/xarm/queeenb_gripper_v2_left.stl" scale="0.001 0.001 0.001"/>
         </geometry>
         <material name="${prefix}Silver"/>
       </visual>
       <collision>
-        <origin xyz="-0.045 -0.048 0.096" rpy="1.5707963267948966 0 -1.5707963267948966"/>
-        <geometry>
-          <mesh filename="${mesh_path}/gripper/xarm/queeenb_gripper_v2_right.stl" scale="0.001 0.001 0.001"/>
+        <origin xyz="0.045 -0.048 0.096" rpy="1.5707963267948966 0 -1.5707963267948966"/>
+        <geometry>
+          <mesh filename="${mesh_path}/gripper/xarm/queeenb_gripper_v2_left.stl" scale="0.001 0.001 0.001"/>
         </geometry>
       </collision>
@@ -161,14 +161,14 @@
         origin_rpy="0 0 0" />
       <visual>
-        <origin xyz="-0.045 0.048 0.096" rpy="1.5707963267948966 0 1.5707963267948966"/>
-        <geometry>
-          <mesh filename="${mesh_path}/gripper/xarm/queeenb_gripper_v2_left.stl" scale="0.001 0.001 0.001"/>
+        <origin xyz="0.045 0.048 0.096" rpy="1.5707963267948966 0 1.5707963267948966"/>
+        <geometry>
+          <mesh filename="${mesh_path}/gripper/xarm/queeenb_gripper_v2_right.stl" scale="0.001 0.001 0.001"/>
         </geometry>
         <material name="${prefix}Silver"/>
       </visual>
       <collision>
-        <origin xyz="-0.045 0.048 0.096" rpy="1.5707963267948966 0 1.5707963267948966"/>
-        <geometry>
-          <mesh filename="${mesh_path}/gripper/xarm/queeenb_gripper_v2_left.stl" scale="0.001 0.001 0.001"/>
+        <origin xyz="0.045 0.048 0.096" rpy="1.5707963267948966 0 1.5707963267948966"/>
+        <geometry>
+          <mesh filename="${mesh_path}/gripper/xarm/queeenb_gripper_v2_right.stl" scale="0.001 0.001 0.001"/>
         </geometry>
       </collision>
